File: Hardware/ATTiny Thing/ATTiny Thing.kicad_pcb (KiCad board)
At the start: 2 copper layers, 30 x 14 mm, 15 parts, among them J1 JST_SH_BM048, J2 UPDI Connection, U1 ATtiny1617

Commit message: Refined the ATTiny Thing
Parts:
- added REF**: DagNabbit, tinker:DagNabbit, B.Cu at (110.0, 100.0)
- G***: moved to B.Cu
- moved G*** 21.4 mm to (89.0, 100.0), turned to 180 degrees
- moved J2 9.29 mm to (99.1, 105.2)
- moved C1 7.37 mm to (89.0, 94.8), turned to 0 degrees
- moved R1 7.08 mm to (97.7, 102.1), turned to 0 degrees
- moved R2 3.71 mm to (100.7, 102.1)
- moved R4 3.45 mm to (95.5, 100.4)
- moved C2 3.41 mm to (102.6, 98.6)
- moved U1 3.40 mm to (99.1, 98.6)
- moved REF** 3.38 mm to (110.0, 100.0)
- moved R3 2.81 mm to (95.5, 97.4)
Connections:
- net SCL renamed PB0
- net SDA renamed PB1
Routing:
- net ~{RESET}: track 8.09 -> 3.11 mm
- net /PA0: track 6.34 -> 2.70 mm
- net PB0: track 8.05 -> 9.98 mm
- net GND: track 6.18 -> 7.87 mm
- net PB1: track 7.64 -> 8.80 mm
Other:
- board text added: "GND 3v3 SDA SCL"
- board text added: "The big question is... What could this little board turn into???"
