File: Hardware/RGB Thing 2/RGB Thing 2.kicad_pcb (KiCad board)
At the start: 2 copper layers, 30 x 14 mm, 16 parts, among them J1 JST_SH_BM048, J2 UPDI Connection, U1 ATtiny1617

Commit message: ...
Parts:
- moved C1 1.00 mm to (88.0, 95.1)
Changed lines of the file:
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@@
   )
   (footprint "Capacitor_SMD:C_0805_2012Metric" (layer "F.Cu")
-    (at 88.9508 94.8436)
+    (at 87.9856 95.0976)
     (descr "Capacitor SMD 0805 (2012 Metric), square (rectangular) end terminal, IPC_7351 nominal, (Body size source: IPC-SM-782 page 76, https://www.pcb-3d.com/wordpress/wp-content/uploads/ipc-sm-782a_amendment_1_and_2.pdf, https://docs.google.com/spreadsheets/d/1BsfQQcO9C6DZCsRaXUlFlo91Tg2WpOkGARC1WS5S8t0/edit?usp=sharing), generated with kicad-footprint-generator")
     (tags "capacitor")
@@
   (gr_arc (start 113 93) (mid 114.414214 93.585786) (end 115 95) (layer "Edge.Cuts") (width 0.05))
   (gr_line (start 85 95) (end 85 105) (layer "Edge.Cuts") (width 0.05))
-  (gr_text "${COMMENT1} (v${REVISION})" (at 97 95.2) (layer "F.SilkS")
+  (gr_text "${COMMENT1} (v${REVISION})" (at 97 95.3) (layer "F.SilkS")
     (effects (font (size 0.75 0.75) (thickness 0.15)))
   )
@@
     (effects (font (size 0.6 0.5) (thickness 0.05)))
   )
+  (segment (start 88.9356 96.9356) (end 90 98) (width 0.2) (layer "F.Cu") (net 1))
   (segment (start 113.174502 101.108497) (end 112.121503 101.108497) (width 0.2) (layer "F.Cu") (net 1))
+  (segment (start 88.9356 95.0976) (end 88.9356 96.9356) (width 0.2) (layer "F.Cu") (net 1))
   (segment (start 112.099871 96.130129) (end 112 96.23) (width 0.2) (layer "F.Cu") (net 1))
   (segment (start 113.174502 96.130129) (end 112.099871 96.130129) (width 0.2) (layer "F.Cu") (net 1))
@@
   (segment (start 97.31 98.8528) (end 97.06 98.6028) (width 0.2) (layer "F.Cu") (net 1))
   (segment (start 100.091 98.8528) (end 100.616 99.3778) (width 0.2) (layer "F.Cu") (net 1))
-  (segment (start 90 98) (end 90 94.9428) (width 0.2) (layer "F.Cu") (net 1))
-  (segment (start 90 94.9428) (end 89.9008 94.8436) (width 0.2) (layer "F.Cu") (net 1))
   (via (at 113.174502 96.130129) (size 0.8) (drill 0.4) (layers "F.Cu" "B.Cu") (net 1))
   (via (at 86.125 102) (size 0.8) (drill 0.4) (layers "F.Cu" "B.Cu") (net 1))
