File: Hardware/USB-C/USB-C.kicad_pcb (KiCad board)
At the start: 2 copper layers, 30 x 14 mm, 4 parts, among them J101 USB_C_Receptacle, J102 USB_C_Receptacle

Commit message: ...
Parts:
- J101, J102: footprint tinker:USB_C_Receptacle_HRO_TYPE-C-NARROW -> tinker:USB_C(sd)
Routing:
- net Vbus: track 68.7 -> 85.9 mm
- net GND: track 5.80 -> 0.00 mm
- net UDb-: track 13.9 -> 15.7 mm
- net UDb+: track 13.9 -> 15.7 mm
- net UDa-: track 13.9 -> 15.7 mm
- net UDa+: track 13.9 -> 15.7 mm
- net SBU2: track 13.9 -> 15.7 mm
- net SBU1: track 13.9 -> 15.7 mm
- net CC2: track 13.9 -> 15.7 mm
- net CC1: track 13.9 -> 15.7 mm
- added copper zone on F.Cu, net GND
- removed copper zone on F.Cu, net Vbus
