File: Hardware/I2C Thing/I2C Thing.kicad_pcb (KiCad board)
At the start: 2 copper layers, 30 x 14 mm, 3 parts, among them J1 JST_SH_BM048

Commit message: ...
Parts:
- added C1: 4.7uF, Capacitor_SMD:C_0805_2012Metric, F.Cu at (88.0, 95.1)
Connections:
- net SCL_ renamed SCL
- net SDA_ renamed SDA
- J1 pad 2: I2C-Vcc_ -> I2C-Vcc
Routing:
- net GND: track 0.00 -> 3.34 mm
- added copper zone on F.Cu, net I2C-Vcc
- removed copper zone on F.Cu, net I2C-Vcc_
Other:
- board text added: "GND 3v3 SDA SCL"
Changed lines of the file:
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@@
   (net 0 "")
   (net 1 "GND")
-  (net 2 "I2C-Vcc_")
-  (net 3 "SDA_")
-  (net 4 "SCL_")
+  (net 2 "I2C-Vcc")
+  (net 3 "SDA")
+  (net 4 "SCL")
   (footprint "tinker:DagNabbit" (layer "F.Cu")
     (at 106 100)
@@
     (property "Sheetname" "")
     (attr smd)
-    (fp_text reference "J1" (at 0 -3.98 90) (layer "F.SilkS")
-      (effects (font (size 1 1) (thickness 0.15)))
+    (fp_text reference "J1" (at -3.5308 0.0144 180) (layer "F.SilkS")
+      (effects (font (size 0.5 0.5) (thickness 0.05)))
     )
     (fp_text value "JST_SH_BM048" (at 0 3.98 90) (layer "F.Fab")
@@
       (net 1 "GND") (pinfunction "Pin_1") (pintype "passive"))
     (pad "2" smd roundrect (at -0.5 -2 270) (size 0.6 1.55) (layers "F.Cu" "F.Paste" "F.Mask") (roundrect_rratio 0.25)
-      (net 2 "I2C-Vcc_") (pinfunction "Pin_2") (pintype "passive"))
+      (net 2 "I2C-Vcc") (pinfunction "Pin_2") (pintype "passive"))
     (pad "3" smd roundrect (at 0.5 -2 270) (size 0.6 1.55) (layers "F.Cu" "F.Paste" "F.Mask") (roundrect_rratio 0.25)
-      (net 3 "SDA_") (pinfunction "Pin_3") (pintype "passive"))
+      (net 3 "SDA") (pinfunction "Pin_3") (pintype "passive"))
     (pad "4" smd roundrect (at 1.5 -2 270) (size 0.6 1.55) (layers "F.Cu" "F.Paste" "F.Mask") (roundrect_rratio 0.25)
-      (net 4 "SCL_") (pinfunction "Pin_4") (pintype "passive"))
+      (net 4 "SCL") (pinfunction "Pin_4") (pintype "passive"))
     (pad "MP" smd roundrect (at 2.8 1.875 270) (size 1.2 1.8) (layers "F.Cu" "F.Paste" "F.Mask") (roundrect_rratio 0.208333)
       (net 1 "GND") (pinfunction "MountPin") (pintype "passive"))
@@
     )
   )
+  (footprint "Capacitor_SMD:C_0805_2012Metric" (layer "F.Cu")
+    (at 87.9856 95.0976)
+    (descr "Capacitor SMD 0805 (2012 Metric), square (rectangular) end terminal, IPC_7351 nominal, (Body size source: IPC-SM-782 page 76, https://www.pcb-3d.com/wordpress/wp-content/uploads/ipc-sm-782a_amendment_1_and_2.pdf, https://docs.google.com/spreadsheets/d/1BsfQQcO9C6DZCsRaXUlFlo91Tg2WpOkGARC1WS5S8t0/edit?usp=sharing), generated with kicad-footprint-generator")
+    (tags "capacitor")
+    (property "LCSC" "C107153")
+    (property "Sheetfile" "I2C Thing.kicad_sch")
+    (property "Sheetname" "")
+    (attr smd)
+    (fp_text reference "C1" (at 0 -1.1176) (layer "F.SilkS")
+      (effects (font (size 0.5 0.5) (thickness 0.05)))
+    )
+    (fp_text value "4.7uF" (at 0 1.68) (layer "F.Fab")
+      (effects (font (size 1 1) (thickness 0.15)))
+    )
+    (fp_text user "${REFERENCE}" (at 0 0) (layer "F.Fab")
+      (effects (font (size 0.5 0.5) (thickness 0.08)))
+    )
+    (fp_line (start -0.261252 0.735) (end 0.261252 0.735) (layer "F.SilkS") (width 0.12))
+    (fp_line (start -0.261252 -0.735) (end 0.261252 -0.735) (layer "F.SilkS") (width 0.12))
+    (fp_line (start 1.7 0.98) (end -1.7 0.98) (layer "F.CrtYd") (width 0.05))
+    (fp_line (start 1.7 -0.98) (end 1.7 0.98) (layer "F.CrtYd") (width 0.05))
+    (fp_line (start -1.7 -0.98) (end 1.7 -0.98) (layer "F.CrtYd") (width 0.05))
+    (fp_line (start -1.7 0.98) (end -1.7 -0.98) (layer "F.CrtYd") (width 0.05))
+    (fp_line (start 1 0.625) (end -1 0.625) (layer "F.Fab") (width 0.1))
+    (fp_line (start 1 -0.625) (end 1 0.625) (layer "F.Fab") (width 0.1))
+    (fp_line (start -1 -0.625) (end 1 -0.625) (layer "F.Fab") (width 0.1))
+    (fp_line (start -1 0.625) (end -1 -0.625) (layer "F.Fab") (width 0.1))
+    (pad "1" smd roundrect (at -0.95 0) (size 1 1.45) (layers "F.Cu" "F.Paste" "F.Mask") (roundrect_rratio 0.25)
+      (net 2 "I2C-Vcc") (pintype "passive"))
+    (pad "2" smd roundrect (at 0.95 0) (size 1 1.45) (layers "F.Cu" "F.Paste" "F.Mask") (roundrect_rratio 0.25)
+      (net 1 "GND") (pintype "passive"))
+    (model "${KICAD6_3DMODEL_DIR}/Capacitor_SMD.3dshapes/C_0805_2012Metric.wrl"
+      (offset (xyz 0 0 0))
+      (scale (xyz 1 1 1))
+      (rotate (xyz 0 0 0))
+    )
+  )
   (gr_line (start 87 107) (end 113 107) (layer "Edge.Cuts") (width 0.05))
   (gr_arc (start 85 95) (mid 85.585786 93.585786) (end 87 93) (layer "Edge.Cuts") (width 0.05))
@@
     (effects (font (size 0.9 0.9) (thickness 0.15)))
   )
+  (gr_text "GND\n3v3\nSDA\nSCL" (at 91.4908 100) (layer "F.SilkS")
+    (effects (font (size 0.6 0.5) (thickness 0.05)))
+  )
   (gr_text "${TITLE}" (at 100 94) (layer "F.SilkS")
     (effects (font (size 0.9 0.9) (thickness 0.15)))
@@
     (effects (font (size 0.9 0.9) (thickness 0.15)))
   )
+  (segment (start 88.9356 95.0976) (end 88.9356 96.9356) (width 0.6) (layer "F.Cu") (net 1))
+  (segment (start 88.9356 96.9356) (end 90 98) (width 0.6) (layer "F.Cu") (net 1))
   (via (at 86.125 102) (size 0.8) (drill 0.4) (layers "F.Cu" "B.Cu") (net 1))
   (via (at 90 98) (size 0.8) (drill 0.4) (layers "F.Cu" "B.Cu") (net 1))
   (via (at 86.125 98) (size 0.8) (drill 0.4) (layers "F.Cu" "B.Cu") (net 1))
-  (zone (net 2) (net_name "I2C-Vcc_") (layer "F.Cu") (hatch edge 0.508)
-    (connect_pads (clearance 0.508))
+  (zone (net 2) (net_name "I2C-Vcc") (layer "F.Cu") (hatch edge 0.508)
+    (connect_pads (clearance 0.254))
     (min_thickness 0.254) (filled_areas_thickness no)
-    (fill yes (thermal_gap 0.508) (thermal_bridge_width 0.508))
+    (fill yes (thermal_gap 0.254) (thermal_bridge_width 0.508))
     (polygon
       (pts
@@
   )
   (zone (net 1) (net_name "GND") (layer "B.Cu") (hatch edge 0.508)
-    (connect_pads (clearance 0.508))
+    (connect_pads (clearance 0.254))
     (min_thickness 0.254) (filled_areas_thickness no)
-    (fill yes (thermal_gap 0.508) (thermal_bridge_width 0.508))
+    (fill yes (thermal_gap 0.254) (thermal_bridge_width 0.508))
     (polygon
       (pts
