File: Hardware/I2C Thing/I2C Thing.kicad_sch (KiCad schematic)
At the start: 1 part, among them J1 JST_SH_BM048

Commit message: ...
Parts:
- added C1: 4.7uF, Capacitor_SMD:C_0805_2012Metric, symbol Device:C
Connections:
- net GND: now also C1.2
- net I2C-Vcc_ renamed I2C-Vcc
- net I2C-Vcc: now also C1.1
- net SCL_ renamed SCL
- net SDA_ renamed SDA
Changed lines of the file:
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@@
     (stroke (width 0) (type default) (color 0 0 0 0))
   )
-  (global_label "SDA_" (shape input) (at 39.37 38.1 180) (fields_autoplaced)
+  (global_label "SDA" (shape input) (at 39.37 38.1 180) (fields_autoplaced)
     (effects (font (size 1.27 1.27)) (justify right))
-    (property "Intersheet References" "${INTERSHEET_REFS}" (id 0) (at 33.5987 38.0206 0)
+    (property "Intersheet References" "${INTERSHEET_REFS}" (id 0) (at 33.3888 38.0206 0)
       (effects (font (size 1.27 1.27)) (justify right) hide)
     )
   )
-  (global_label "I2C-Vcc_" (shape input) (at 39.37 35.56 180) (fields_autoplaced)
+  (global_label "I2C-Vcc" (shape input) (at 80.01 38.1 180) (fields_autoplaced)
     (effects (font (size 1.27 1.27)) (justify right))
-    (property "Intersheet References" "${INTERSHEET_REFS}" (id 0) (at 28.1558 35.4806 0)
+    (property "Intersheet References" "${INTERSHEET_REFS}" (id 0) (at 69.6745 38.0206 0)
       (effects (font (size 1.27 1.27)) (justify right) hide)
     )
   )
-  (global_label "SCL_" (shape input) (at 39.37 40.64 180) (fields_autoplaced)
+  (global_label "I2C-Vcc" (shape input) (at 39.37 35.56 180) (fields_autoplaced)
     (effects (font (size 1.27 1.27)) (justify right))
-    (property "Intersheet References" "${INTERSHEET_REFS}" (id 0) (at 33.5987 40.5606 0)
+    (property "Intersheet References" "${INTERSHEET_REFS}" (id 0) (at 29.0345 35.4806 0)
+      (effects (font (size 1.27 1.27)) (justify right) hide)
+    )
+  )
+  (global_label "SCL" (shape input) (at 39.37 40.64 180) (fields_autoplaced)
+    (effects (font (size 1.27 1.27)) (justify right))
+    (property "Intersheet References" "${INTERSHEET_REFS}" (id 0) (at 33.4493 40.5606 0)
       (effects (font (size 1.27 1.27)) (justify right) hide)
     )
@@
     (pin "1")
   )
+  (symbol (lib_id "Device:C") (at 80.01 41.91 0) (unit 1)
+    (in_bom yes) (on_board yes) (fields_autoplaced)
+    (property "Reference" "C1" (id 0) (at 83.82 40.6399 0)
+      (effects (font (size 1.27 1.27)) (justify left))
+    )
+    (property "Value" "4.7uF" (id 1) (at 83.82 43.1799 0)
+      (effects (font (size 1.27 1.27)) (justify left))
+    )
+    (property "Footprint" "Capacitor_SMD:C_0805_2012Metric" (id 2) (at 80.9752 45.72 0)
+      (effects (font (size 1.27 1.27)) hide)
+    )
+    (property "Datasheet" "~" (id 3) (at 80.01 41.91 0)
+      (effects (font (size 1.27 1.27)) hide)
+    )
+    (property "LCSC" "C107153" (id 4) (at 80.01 41.91 0)
+      (effects (font (size 1.27 1.27)) hide)
+    )
+    (pin "1")
+    (pin "2")
+  )
   (symbol (lib_id "power:GND") (at 27.94 45.72 0) (unit 1)
     (in_bom yes) (on_board yes)
@@
     )
     (property "Datasheet" "" (id 3) (at 27.94 45.72 0)
+      (effects (font (size 1.27 1.27)) hide)
+    )
+    (pin "1")
+  )
+  (symbol (lib_id "power:GND") (at 80.01 45.72 0) (unit 1)
+    (in_bom yes) (on_board yes) (fields_autoplaced)
+    (property "Reference" "#PWR0103" (id 0) (at 80.01 52.07 0)
+      (effects (font (size 1.27 1.27)) hide)
+    )
+    (property "Value" "GND" (id 1) (at 80.01 50.8 0))
+    (property "Footprint" "" (id 2) (at 80.01 45.72 0)
+      (effects (font (size 1.27 1.27)) hide)
+    )
+    (property "Datasheet" "" (id 3) (at 80.01 45.72 0)
       (effects (font (size 1.27 1.27)) hide)
     )
@@
       (reference "#PWR0102") (unit 1) (value "GND") (footprint "")
     )
+    (path "/71b0d8fb-0c75-45a3-966e-b30cd0e49f17"
+      (reference "#PWR0103") (unit 1) (value "GND") (footprint "")
+    )
+    (path "/2735e39d-7d89-4596-b1d0-dff1f5a44b7c"
+      (reference "C1") (unit 1) (value "4.7uF") (footprint "Capacitor_SMD:C_0805_2012Metric")
+    )
     (path "/bbc4fe36-8875-4a27-a8db-dd1d51bc6d7a"
